Commit message: change the rotation axis of the caster wheel

File: description/urdf/pioneer3dx.urdf (robot description, URDF)
Before this commit: robot pioneer3dx, 11 links, 10 joints
Joints:
- joint base_caster_swivel_joint: axis (none) -> 0 0 1

File: description/urdf/pioneer3dx.urdf.xacro (robot description, xacro)
@@ -111,4 +111,5 @@
 	<joint name="base_caster_swivel_joint" type="continuous">
 		<origin xyz="-0.185 0 0.055" rpy="0 0 0"/>
+		<axis xyz="0 0 1"/>
 		<anchor xyz="0 0 0"/>
     	<limit effort="100" velocity="100" k_velocity="0" />
